Commit message: fix(robots,launch)!: standardise OpenArm on one wire naming convention
BREAKING CHANGE: `robots/openarm/openarm.urdf` now spells joints and links as
upstream does (`openarm_left_joint1`, `openarm_left_base_link`) instead of the
stripped `left_joint1` / `left_base_link`. Anything reading that file by link or
joint name must use the new spelling. The manifest's logical joint names are
unchanged.

What changed
- `robots/openarm/openarm.urdf`: 108 distinct names re-prefixed (325 attribute
  sites). Rename only — no geometry, no joint added or removed. Verified name-set
  equality against the rig's own `xacro` output for the pinned
  `openarm_description` SHA, rendered with the mappings `openarm.bimanual.launch.py`
  uses; the only names not present upstream are two `<hardware>` `<param>`s.
- `openral_cli.robot._RENAME` is now empty: openarm's `"openarm_` → `"` strip is
  gone, so re-vendoring cannot reintroduce the divergence.
- `deploy_e2e.launch.py` remaps the graph's `robot_state_publisher` off
  `/robot_description` onto `/openral/robot_description` whenever a vendor
  bringup is included; `/openral/robot_description` joins the Foxglove
  allowlist.
- Corrects a claim I put in this file earlier: the two robot_state_publishers
  were *not* harmlessly additive.

Why
Both descriptions come from the same Enactic repo and the same xacro — we
renamed one on the way in, to match the manifest's logical joint names. That
left the vendored URDF as the only artefact spelling this robot differently: its
ros2_control graph, `/joint_states`, MJCF and
`OpenArmRealHAL.ros2_control_joint_names()` all say `openarm_left_joint1`.

Two spellings broke two things, both silently. `joint_state_broadcaster`'s
`use_urdf_to_filter` publishes only joints the robot description also names, so
a disjoint intersection yields `name: []` at 741 Hz with every controller active
and the CAN bus healthy — measured on the cell: 7317 empty messages, 0
populated, while the same bringup launched alone published all 16 joints. And
`robot_state_publisher` poses its tree by matching those names, so the whole arm
sat at the rest pose in `/tf`, placing every arm-mounted sensor as if the robot
had never moved.

The remap is what the matching names then make load-bearing rather than
optional: `controller_manager` reads `/robot_description` on Jazzy, and the
manifest URDF declares `mock_components/GenericSystem` where the vendor declares
`openarm_hardware/OpenArmHW`. Now that both descriptions are name-compatible, a
controller_manager latching ours would come up on mock hardware — controllers
active, `/joint_states` plausible, arm motionless. Sharing that topic was never
safe; it was only ever visibly broken.

The manifest's logical joint names (`left_joint1`) stay: they are the
action-vector contract, shared with other robots and pinned by published rSkill
manifests (`rskills/rskill-pi05-openarm-restock_shelf-bf16`). `sim_joint_name`
and `ros2_control_joint_names()` are the declared bridges, now test-pinned.

How tested
`tests/unit/test_openarm_wire_names.py` — no stripped joint survives; the URDF
declares every joint the real HAL reads; `<ros2_control>` joints are a subset of
URDF joints (the set `use_urdf_to_filter` intersects); every `sim_joint_name`
reaches a real URDF joint. `test_urdf_root_frame_bridge` updated for the new
link names — the 0.698 m bridge is unchanged. `just lint`, `mypy --strict`,
markers clean; full unit + sim/safety + hal + cli + foxglove sweep green apart
from a pre-existing order-dependent failure in `test_sim_attached_hal.py`.

Co-Authored-By: Claude Opus 5 (1M context) <noreply@anthropic.com>
Claude-Session: https://claude.ai/code/session_01EH1WdGYp6qmRm4rdZ29eVQ
Signed-off-by: Adrian <adrianllopart@gmail.com>

File: robots/openarm/openarm.urdf (robot description, URDF)
Before this commit: robot v20, 22 links, 21 joints
Links:
- removed link body_link0
- removed link left_base_link
- removed link left_ee_base_link
- removed link left_ee_link1
- removed link left_ee_link2
- removed link left_link1
- removed link left_link2
- removed link left_link3
- removed link left_link4
- removed link left_link5
- removed link left_link6
- removed link right_base_link
- removed link right_ee_base_link
- removed link right_ee_link1
- removed link right_ee_link2
- removed link right_link1
- removed link right_link2
- removed link right_link3
- removed link right_link4
- removed link right_link5
- removed link right_link6
- added link openarm_body_link0, mass 13.89; collision mesh filename=package://openarm_description/assets/robot/openarm_v2.0/mes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 scale=0.001 0.001 0.001; visual mesh filename=package://openarm_description/assets/robot/openarm_v2.0/mes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 scale=0.001 0.001 0.001
- added link openarm_left_base_link, mass 0.487784887988258; collision mesh filename=package://openarm_description/assets/robot/openarm_v2.0/mes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 scale=1 -1 1; visual mesh filename=package://openarm_description/assets/robot/openarm_v2.0/mes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 scale=1 -1 1
- added link openarm_left_ee_base_link, mass 0.52832; collision mesh filename=package://openarm_description/assets/end_effector/pinch_gri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 scale=1 -1 1; visual mesh filename=package://openarm_description/assets/end_effector/pinch_gri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 scale=1 -1 1
- added link openarm_left_ee_link1, mass 0.125979047366671; collision mesh filename=package://openarm_description/assets/end_effector/pinch_gri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 scale=1 -1 1; visual mesh filename=package://openarm_description/assets/end_effector/pinch_gri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 scale=1 -1 1
- added link openarm_left_ee_link2, mass 0.11372; collision mesh filename=package://openarm_description/assets/end_effector/pinch_gri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 scale=1 -1 1; visual mesh filename=package://openarm_description/assets/end_effector/pinch_gri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 scale=1 -1 1
- added link openarm_left_link1, mass 0.561428544234246; collision mesh filename=package://openarm_description/assets/robot/openarm_v2.0/mes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 scale=1 -1 1; visual mesh filename=package://openarm_description/assets/robot/openarm_v2.0/mes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 scale=1 -1 1
- added link openarm_left_link2, mass 0.295592749115978; collision mesh filename=package://openarm_description/assets/robot/openarm_v2.0/mes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 scale=1 -1 1; visual mesh filename=package://openarm_description/assets/robot/openarm_v2.0/mes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 scale=1 -1 1
- added link openarm_left_link3, mass 0.850916861288263; collision mesh filename=package://openarm_description/assets/robot/openarm_v2.0/mes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 scale=1 1 1; visual mesh filename=package://openarm_description/assets/robot/openarm_v2.0/mes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 scale=1 1 1
- added link openarm_left_link4, mass 0.590845933035621; collision mesh filename=package://openarm_description/assets/robot/openarm_v2.0/mes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 scale=1 1 1; visual mesh filename=package://openarm_description/assets/robot/openarm_v2.0/mes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 scale=1 1 1
- added link openarm_left_link5, mass 0.5803968030561; collision mesh filename=package://openarm_description/assets/robot/openarm_v2.0/mes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 scale=1 -1 1; visual mesh filename=package://openarm_description/assets/robot/openarm_v2.0/mes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 scale=1 -1 1
- added link openarm_left_link6, mass 0.368168327082267; collision mesh filename=package://openarm_description/assets/robot/openarm_v2.0/mes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 scale=1 -1 1; visual mesh filename=package://openarm_description/assets/robot/openarm_v2.0/mes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 scale=1 -1 1
- added link openarm_right_base_link, mass 0.487784887988258; collision mesh filename=package://openarm_description/assets/robot/openarm_v2.0/mes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 scale=1 1 1; visual mesh filename=package://openarm_description/assets/robot/openarm_v2.0/mes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 scale=1 1 1
- added link openarm_right_ee_base_link, mass 0.52832; collision mesh filename=package://openarm_description/assets/end_effector/pinch_gri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 scale=1 1 1; visual mesh filename=package://openarm_description/assets/end_effector/pinch_gri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 scale=1 1 1
- added link openarm_right_ee_link1, mass 0.125979047366671; collision mesh filename=package://openarm_description/assets/end_effector/pinch_gri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 scale=1 1 1; visual mesh filename=package://openarm_description/assets/end_effector/pinch_gri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 scale=1 1 1
- added link openarm_right_ee_link2, mass 0.11372; collision mesh filename=package://openarm_description/assets/end_effector/pinch_gri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 scale=1 1 1; visual mesh filename=package://openarm_description/assets/end_effector/pinch_gri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 scale=1 1 1
- added link openarm_right_link1, mass 0.561428544234246; collision mesh filename=package://openarm_description/assets/robot/openarm_v2.0/mes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 scale=1 1 1; visual mesh filename=package://openarm_description/assets/robot/openarm_v2.0/mes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 scale=1 1 1
- added link openarm_right_link2, mass 0.295592749115978; collision mesh filename=package://openarm_description/assets/robot/openarm_v2.0/mes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 scale=1 1 1; visual mesh filename=package://openarm_description/assets/robot/openarm_v2.0/mes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 scale=1 1 1
- added link openarm_right_link3, mass 0.850916861288263; collision mesh filename=package://openarm_description/assets/robot/openarm_v2.0/mes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 scale=1 1 1; visual mesh filename=package://openarm_description/assets/robot/openarm_v2.0/mes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 scale=1 1 1
- added link openarm_right_link4, mass 0.590845933035621; collision mesh filename=package://openarm_description/assets/robot/openarm_v2.0/mes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 scale=1 1 1; visual mesh filename=package://openarm_description/assets/robot/openarm_v2.0/mes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 scale=1 1 1
- added link openarm_right_link5, mass 0.5803968030561; collision mesh filename=package://openarm_description/assets/robot/openarm_v2.0/mes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 scale=1 1 1; visual mesh filename=package://openarm_description/assets/robot/openarm_v2.0/mes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 scale=1 1 1
- added link openarm_right_link6, mass 0.368168327082267; collision mesh filename=package://openarm_description/assets/robot/openarm_v2.0/mes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 scale=1 1 1; visual mesh filename=package://openarm_description/assets/robot/openarm_v2.0/mes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 scale=1 1 1
Joints:
- removed joint body_link0_mount_joint
- removed joint left_base_link_mount_joint
- removed joint left_finger_joint1
- removed joint left_finger_joint2
- removed joint left_joint1
- removed joint left_joint2
- removed joint left_joint3
- removed joint left_joint4
- removed joint left_joint5
- removed joint left_joint6
- removed joint left_joint7
- removed joint right_base_link_mount_joint
- removed joint right_finger_joint1
- removed joint right_finger_joint2
- removed joint right_joint1
- removed joint right_joint2
- removed joint right_joint3
- removed joint right_joint4
- removed joint right_joint5
- removed joint right_joint6
- removed joint right_joint7
- added joint openarm_body_link0_mount_joint: type fixed, parent world, child openarm_body_link0, origin xyz=0.0 0.0 0.0 rpy=0.0 0.0 0.0
- added joint openarm_left_base_link_mount_joint: type fixed, parent openarm_body_link0, child openarm_left_base_link, origin xyz=0.0 0.031 0.698 rpy=0.0 0.0 0.0
- added joint openarm_left_finger_joint1: type revolute, parent openarm_left_ee_base_link, child openarm_left_ee_link1, origin xyz=-0.0014300000000005003 -0.0180000000000009 -0.0680000000000174 rpy=0.0 -0.0 0.0, axis -1 0 0, limit lower=-1.5708 upper=0 effort=7 velocity=5
- added joint openarm_left_finger_joint2: type revolute, parent openarm_left_ee_base_link, child openarm_left_ee_link2, origin xyz=-0.0014300000000005003 0.0180000000000012 -0.0680000000000215 rpy=0.0 -0.0 0.0, axis -1 0 0, limit lower=0 upper=1.5708 effort=7 velocity=5, mimic joint=openarm_left_finger_joint1 multiplier=-1 offset=0
- added joint openarm_left_joint1: type revolute, parent openarm_left_base_link, child openarm_left_link1, origin xyz=0 0.0625 0 rpy=0 0 0, axis 0 1 0, limit lower=-3.4907 upper=1.3963 effort=40 velocity=16.755
- added joint openarm_left_joint2: type revolute, parent openarm_left_link1, child openarm_left_link2, origin xyz=0 0.0600000000000001 0 rpy=0 0 0, axis -1 0 0, limit lower=-3.3161 upper=0.17453 effort=40 velocity=16.755
- added joint openarm_left_joint3: type revolute, parent openarm_left_link2, child openarm_left_link3, origin xyz=0 0 -0.0662500000000008 rpy=0 0 0, axis 0 0 -1, limit lower=-1.5708 upper=1.5708 effort=27 velocity=5.4454
- added joint openarm_left_joint4: type revolute, parent openarm_left_link3, child openarm_left_link4, origin xyz=0 0 -0.15375 rpy=0 0 0, axis 0 -1 0, limit lower=0 upper=2.4435 effort=27 velocity=5.4454
- added joint openarm_left_joint5: type revolute, parent openarm_left_link4, child openarm_left_link5, origin xyz=0 0 -0.0955000000000005 rpy=0 0 0, axis 0 0 -1, limit lower=-1.5708 upper=1.5708 effort=7 velocity=20.944
- added joint openarm_left_joint6: type revolute, parent openarm_left_link5, child openarm_left_link6, origin xyz=0 0 -0.120499999999998 rpy=0 0 0, axis 0 -1 0, limit lower=-0.7854 upper=0.7854 effort=7 velocity=20.944
- added joint openarm_left_joint7: type revolute, parent openarm_left_link6, child openarm_left_ee_base_link, origin xyz=0 0 0 rpy=0 0 0, axis 1 0 0, limit lower=-0.7854 upper=0.7854 effort=7 velocity=20.944
- added joint openarm_right_base_link_mount_joint: type fixed, parent openarm_body_link0, child openarm_right_base_link, origin xyz=0.0 -0.031 0.698 rpy=0.0 0.0 0.0
- added joint openarm_right_finger_joint1: type revolute, parent openarm_right_ee_base_link, child openarm_right_ee_link1, origin xyz=-0.0014300000000005003 0.0180000000000009 -0.0680000000000174 rpy=0.0 -0.0 0.0, axis -1 0 0, limit lower=-1.5708 upper=0 effort=7 velocity=5
- added joint openarm_right_finger_joint2: type revolute, parent openarm_right_ee_base_link, child openarm_right_ee_link2, origin xyz=-0.0014300000000005003 -0.0180000000000012 -0.0680000000000215 rpy=0.0 -0.0 0.0, axis -1 0 0, limit lower=0 upper=1.5708 effort=7 velocity=5, mimic joint=openarm_right_finger_joint1 multiplier=-1 offset=0
- added joint openarm_right_joint1: type revolute, parent openarm_right_base_link, child openarm_right_link1, origin xyz=0 -0.0625 0 rpy=0 0 0, axis 0 -1 0, limit lower=-1.3963 upper=3.4907 effort=40 velocity=16.755
- added joint openarm_right_joint2: type revolute, parent openarm_right_link1, child openarm_right_link2, origin xyz=0 -0.0600000000000001 0 rpy=0 0 0, axis -1 0 0, limit lower=-0.17453 upper=3.3161 effort=40 velocity=16.755
- added joint openarm_right_joint3: type revolute, parent openarm_right_link2, child openarm_right_link3, origin xyz=0 0 -0.0662500000000008 rpy=0 0 0, axis 0 0 -1, limit lower=-1.5708 upper=1.5708 effort=27 velocity=5.4454
- added joint openarm_right_joint4: type revolute, parent openarm_right_link3, child openarm_right_link4, origin xyz=0 0 -0.15375 rpy=0 0 0, axis 0 -1 0, limit lower=0 upper=2.4435 effort=27 velocity=5.4454
- added joint openarm_right_joint5: type revolute, parent openarm_right_link4, child openarm_right_link5, origin xyz=0 0 -0.0955000000000005 rpy=0 0 0, axis 0 0 -1, limit lower=-1.5708 upper=1.5708 effort=7 velocity=20.944
- added joint openarm_right_joint6: type revolute, parent openarm_right_link5, child openarm_right_link6, origin xyz=0 0 -0.120499999999998 rpy=0 0 0, axis 0 1 0, limit lower=-0.7854 upper=0.7854 effort=7 velocity=20.944
- added joint openarm_right_joint7: type revolute, parent openarm_right_link6, child openarm_right_ee_base_link, origin xyz=0 0 0 rpy=0 0 0, axis 1 0 0, limit lower=-0.7854 upper=0.7854 effort=7 velocity=20.944

Commit message: fix(sim): open the OpenArm's left jaw outward in Isaac
The vendored OpenArm URDF mirrors the left hand's finger meshes
(scale 1 -1 1) and hinge origins but keeps the right hand's limits
(finger_joint1 [-1.5708, 0]). On the shared -x hinge axis the left jaw opens
positive, as in the MJCF ([0, 0.7854]) and the manifest's left_gripper range,
so upstream's limits allow only an inward swing. The Isaac gripper spec
picked the passthrough sign from those limits and negated the left jaw's
command to fit them: the left fingers opened crossed, through each other, and
a close swept them back across the object. In the warehouse pick trials the
left jaw never settled, dragged the hand 2.3 cm sideways and the brick slid
out on the lift, while the right hand held every time.

- robots/openarm/openarm.urdf: the left fingers' limits on the opening side
  (finger_joint1 [0, 1.5708], finger_joint2 [-1.5708, 0]); README lists it as
  a vendored deviation.
- _gripper_spec(passthrough): write the manifest's physical value unchanged
  on the URDF axis; a range outside the URDF limits is a ROSConfigError
  instead of a silent negation.
- test: each finger's open target swings it away from the jaw centre (fails
  on the old URDF and spec for the left hand).

The MuJoCo twin, the real hardware and the kernel's collision model (lowered
from the MJCF) never read these limits and are unchanged.

Co-Authored-By: Claude Opus 5.5 <noreply@anthropic.com>
Claude-Session: https://claude.ai/code/session_01KTrV7z7yWp6QksMj6bfNMx
Signed-off-by: Adrian <adrianllopart@gmail.com>

File: robots/openarm/openarm.urdf (robot description, URDF)
Before this commit: robot openarm_v20, 22 links, 21 joints
Joints:
- joint openarm_left_finger_joint1: limit lower=-1.5708 upper=0 effort=7 velocity=5 -> lower=0 upper=1.5708 effort=7 velocity=5
- joint openarm_left_finger_joint2: limit lower=0 upper=1.5708 effort=7 velocity=5 -> lower=-1.5708 upper=0 effort=7 velocity=5

Commit message: fix(robots): refresh the vendored OpenArm arm-link inertials to upstream nominal
The vendored URDF carried stale inertials for base_link and link1-6 of both
arms (base 0.49 kg, link1 0.56, link3 0.85, link6 0.37) where upstream
enactic/openarm_description v2.0 nominal, the v2 MJCF and the real v20
bringup all have 1.14 / 1.14 / 1.07 / 0.48 kg (same CoMs; finger and body
masses already matched). Masses and inertia tensors are now upstream's,
keeping the left arm's mirrored ixy/iyz signs. Gravity torque in the Isaac
and ros2_control paths was ~25 % low in the distal links.

Co-Authored-By: Claude Fable 5.1 <noreply@anthropic.com>
Claude-Session: https://claude.ai/code/session_01SmasLK69CY88zVH9nRMqEJ
Signed-off-by: Adrian <adrianllopart@gmail.com>

File: robots/openarm/openarm.urdf (robot description, URDF)
Before this commit: robot openarm_v20, 22 links, 21 joints
Links:
- link openarm_left_base_link: mass 0.487784887988258 -> 1.1432284943239561
- link openarm_left_link1: mass 0.561428544234246 -> 1.1416684646202298
- link openarm_left_link2: mass 0.295592749115978 -> 0.2775092746011571
- link openarm_left_link3: mass 0.850916861288263 -> 1.073863338202347
- link openarm_left_link4: mass 0.590845933035621 -> 0.6348534566833373
- link openarm_left_link5: mass 0.5803968030561 -> 0.6156588026168502
- link openarm_left_link6: mass 0.368168327082267 -> 0.475202773187987
- link openarm_right_base_link: mass 0.487784887988258 -> 1.1432284943239561
- link openarm_right_link1: mass 0.561428544234246 -> 1.1416684646202298
- link openarm_right_link2: mass 0.295592749115978 -> 0.2775092746011571
- link openarm_right_link3: mass 0.850916861288263 -> 1.073863338202347
- link openarm_right_link4: mass 0.590845933035621 -> 0.6348534566833373
- link openarm_right_link5: mass 0.5803968030561 -> 0.6156588026168502
- link openarm_right_link6: mass 0.368168327082267 -> 0.475202773187987
