Commit message: feat(deploy): real-hardware OpenArm bench scene, HIL gate, and the fixes that let a Hub VLA dispatch on it (#289)
* fix(tools): guard grasp_declaration and vision_attachment in the matrix

_SCENE_SAFETY_KEYS covered place_declaration but not grasp_declaration,
which grants the same kind of kernel exemption, and runtime keys omitted
vision_attachment, whose enabled flag arms the attached-payload check and
whose tf_frames pick the link a payload rides. A round could move either
in a materialised scene unnoticed. (runtime.grasp_allowance_enabled was
already guarded.)

Co-Authored-By: Claude Opus 5.5 <noreply@anthropic.com>
Signed-off-by: Adrian <adrianllopart@gmail.com>

* fix(docs): refresh the drifted compose_so100_runtime line marker

Pre-existing on the base commit: tools/refresh_methods_linenos.py --check
reported 11-ros2-nodes.md stale by one marker.

Co-Authored-By: Claude Opus 5.5 <noreply@anthropic.com>
Signed-off-by: Adrian <adrianllopart@gmail.com>

* docs(methods): merge the duplicated vision_attachment_bridge entries

01-hal.md listed the module's symbols twice with disagreeing contents:
one copy had the release window, the other the place-fixture leg. One
complete section now carries both.

Co-Authored-By: Claude Opus 5.5 <noreply@anthropic.com>
Signed-off-by: Adrian <adrianllopart@gmail.com>

* fix(hal): lift the sim grasp region one voxel off its support

The real producer (_grasp_target.target_region_from_mask, HZ-01xx-6)
puts a grasp region's lower face at support_z + resolution so the
support's cells stay outside it and the kernel still stops fingers at
the table under the target. The sim producer used the target's raw
subtree box, so the twin exempted support-layer cells real would not.

lift_region_off_support shrinks the body-frame box's face on the axis
closest to base +z so its lowest point rises exactly one voxel (the real
rule verbatim for an upright target; None when the target is no taller
than a voxel). The resolution comes from the last /openral/world_voxels
grid via SimSensorBridge._fill_grasp_declaration -> set_voxel_resolution;
before any grid the declaration rides region-less (fail closed). Kept
local rather than shared with _grasp_target, which fits a
gravity-aligned box from a cloud.

The grasp-pair twin now grasps 50 mm over the table instead of 30 mm:
with the bottom block layer no longer exempt, the open pads must clear
it by the 20 mm margin, as they would on real.

Co-Authored-By: Claude Opus 5.5 <noreply@anthropic.com>
Signed-off-by: Adrian <adrianllopart@gmail.com>

* fix(hal): measure the grasp target's support plane from the voxel map

The pre-grasp target producer stood the region's lower face on the search
box's bottom face. That box is a lifted detection bbox whose min-z can sit
below the real table top, which put table cells inside the exemption region
(HZ-01xx-6). The support is now measured: the densest occupied layer in a
column under the search box (reaching 0.15 m below its bottom), and that
layer must also hold cells within 0.10 m of the seed. No such layer is a
typed `no_support` refusal and no region.

Co-Authored-By: Claude Opus 5.5 <noreply@anthropic.com>
Claude-Session: https://claude.ai/code/session_01KTrV7z7yWp6QksMj6bfNMx
Signed-off-by: Adrian <adrianllopart@gmail.com>

* fix(hal): treat a grasp re-fit shrunk inside the held region as occlusion

As the hand closes in it occludes part of the target, so the re-fit shrinks
and shifts. The leg classed that as `target_moved` / `map_disagrees` and
retracted the region at once, instead of freezing it under the lost-view TTL.
A re-fit that fails the map or tracking gate but lies inside the held region
grown by one voxel (`region_within`) is now `occluded_refit`, a lost view: the
held region stays under its freeze TTL and is never replaced by the partial
fit. A re-fit reaching outside it still retracts.

Co-Authored-By: Claude Opus 5.5 <noreply@anthropic.com>
Claude-Session: https://claude.ai/code/session_01KTrV7z7yWp6QksMj6bfNMx
Signed-off-by: Adrian <adrianllopart@gmail.com>

* fix(hal): refuse SegmentInView masks captured off their depth frame

The segmenter stamps each mask with the RGB frame it captured, but neither
the attachment bridge nor the grasp-target leg compared that stamp with the
depth frame the mask is back-projected through, so a mask from one instant
could be laid on depth from another. `mask_depth_skew_reason` now refuses a
reply when any mask is more than `mask_depth_max_skew_s` (default 0.1 s, HAL
param `vision_attachment_mask_depth_max_skew_s`) from that depth frame: a
typed, logged `GRIPPER_FORCE` fallback in the attachment path and a
`mask_depth_skew` lost view in the grasp-target leg.

Co-Authored-By: Claude Opus 5.5 <noreply@anthropic.com>
Claude-Session: https://claude.ai/code/session_01KTrV7z7yWp6QksMj6bfNMx
Signed-off-by: Adrian <adrianllopart@gmail.com>

* fix(hal): take the producer legs' grid age and release bounds from the deploy

The grasp-target and place-fixture legs each hard-coded the real OpenArm
cell's 1.0 s kernel voxel deadline as their grid age bound, the grasp
freeze defaulted to 2 s on the same assumption, and release_clear_m baked
in that cell's 20 mm margin + 20 mm voxel. `VisionAttachmentConfig` now
carries `grid_max_age_s` (used by both legs), `grasp_target_freeze_s`
defaults to twice it, and the cell values remain only as documented
fallbacks. The HAL node declares `vision_attachment_grid_max_age_s`,
`vision_attachment_release_clear_m` and `vision_attachment_release_timeout_s`
for the deploy to set from the kernel's `world_voxel_deadline_s` and margin
+ resolution; `vision_attachment_grasp_target_freeze_s` 0 now means derive.

Co-Authored-By: Claude Opus 5.5 <noreply@anthropic.com>
Claude-Session: https://claude.ai/code/session_01KTrV7z7yWp6QksMj6bfNMx
Signed-off-by: Adrian <adrianllopart@gmail.com>

* fix(reasoner): make the grounded grasp search box a search hint, padded downward too

The docstring claimed the lifted box's bottom (the lowest occupied cell centre in the
detection's frustum) "errs upward (safe) either way"; it does not — table cells caught by
a loose pixel box put it below the support. The box now carries no support semantics (the
HAL producer measures the support layer from the voxel map) and is padded by one voxel +
extrinsic error on every side, downward included, so the support layer is inside it for
the producer to find, and bounded so it reaches no further.

Co-Authored-By: Claude Opus 5.5 <noreply@anthropic.com>
Claude-Session: https://claude.ai/code/session_01KTrV7z7yWp6QksMj6bfNMx
Signed-off-by: Adrian <adrianllopart@gmail.com>

* fix(reasoner): refuse an unnamed gripper on a multi-gripper robot

An empty GraspTargetRef.contact_links defaulted to every role: gripper child link, so on
the bimanual OpenArm one grasp declared both hands and the kernel exemption would let the
idle hand touch the target too. With more than one gripper the grounding now refuses
(ROSReasonerInvalidPlan naming the choices, reported to the LLM); a single-gripper robot
keeps its one link as the default. No rSkill manifest field says which arm a skill drives,
so there is nothing to derive the hand from. The direct-dispatch fixture scene names one
hand; the LLM-facing field description says the same.

Co-Authored-By: Claude Opus 5.5 <noreply@anthropic.com>
Claude-Session: https://claude.ai/code/session_01KTrV7z7yWp6QksMj6bfNMx
Signed-off-by: Adrian <adrianllopart@gmail.com>

* fix(hal): declare the vision attachment effort thresholds the deploy forwards

deploy_sim forwards runtime.vision_attachment.attach_effort / release_effort as HAL params
vision_attachment_attach_effort / _release_effort, which the HAL never declared, so rclpy
dropped them silently and the trigger ran on its default fractions. The HAL now declares
both (0.0 = unset) and passes vision_attachment_trigger_config to the bridge, which turns
the absolute efforts into fractions of the one effort_limit every gripper shares. A live
test loads the params file the CLI writes into the real ManifestHALLifecycleNode and
requires every forwarded vision_attachment_* name declared and the scene's thresholds on
the real GripperEffortTrigger.

Co-Authored-By: Claude Opus 5.5 <noreply@anthropic.com>
Claude-Session: https://claude.ai/code/session_01KTrV7z7yWp6QksMj6bfNMx
Signed-off-by: Adrian <adrianllopart@gmail.com>

* fix(cli): forward the vision producer toggles and refuse an unproduced grasp allowance

Nothing in DeployRuntime mapped the HAL's vision_attachment_grasp_target_enabled /
_place_fixture_enabled, so a scene could not turn either producer on. They are now
VisionAttachmentRuntime fields (default false) forwarded as those HAL params; with the
place leg on, the selected robot unit rides as vision_attachment_robot_unit (the scene's
robot_unit is not in the HAL's environment). deploy run refuses grasp_allowance_enabled
unless the leg and its grasp_target_enabled are on: on real the target leg is the only
region producer, so the kernel would arm the exemption with nothing measuring the region.
deploy sim keeps it (the MuJoCo evidence tracker produces the region).

Co-Authored-By: Claude Opus 5.5 <noreply@anthropic.com>
Claude-Session: https://claude.ai/code/session_01KTrV7z7yWp6QksMj6bfNMx
Signed-off-by: Adrian <adrianllopart@gmail.com>

* fix(cli): derive the vision release-window bounds from the kernel's voxel path

The HAL's release window and grid-age bound read the voxel path the kernel checks. With the
vision leg on, deploy_e2e.launch.py now gives the HAL vision_attachment_grid_max_age_s = the
kernel's world_voxel_deadline_s and vision_attachment_release_clear_m = the kernel's world
margin + one octree cell, from the launch's own _world_voxel_margin_m / _octomap_resolution
(listed before the CLI's params file, so an explicit --hal value still wins). The release
timeout is a calibration point, so it is a scene field (runtime.vision_attachment.
release_timeout_s, default 3.0) forwarded as vision_attachment_release_timeout_s. The HAL
declarations land with the release-window change on the pick/place branch; the live
params test lists release_timeout_s as pending until then.

Co-Authored-By: Claude Opus 5.5 <noreply@anthropic.com>
Claude-Session: https://claude.ai/code/session_01KTrV7z7yWp6QksMj6bfNMx
Signed-off-by: Adrian <adrianllopart@gmail.com>

* fix(reasoner): pad grounded grasp targets by the deploy's octree cell

grasp_target_voxel_m defaulted to REAL_WORLD_VOXEL_MARGIN_M, the kernel's world margin,
which only equals the real 20 mm cell by coincidence (sim maps at 15 mm, and
OPENRAL_OCTOMAP_RESOLUTION_M moves both). deploy_e2e now passes the reasoner
_octomap_resolution(hal_mode), the same value octomap_server gets; the standalone default
is the real 20 mm cell, stated as such.

Co-Authored-By: Claude Opus 5.5 <noreply@anthropic.com>
Claude-Session: https://claude.ai/code/session_01KTrV7z7yWp6QksMj6bfNMx
Signed-off-by: Adrian <adrianllopart@gmail.com>

* test(hal): require every forwarded vision param to be declared, release timeout included

The HAL now declares vision_attachment_release_timeout_s, so the live params
test drops its pending-declaration exemption.

Co-Authored-By: Claude Opus 5.5 <noreply@anthropic.com>
Claude-Session: https://claude.ai/code/session_01KTrV7z7yWp6QksMj6bfNMx
Signed-off-by: Adrian <adrianllopart@gmail.com>

* docs(methods): refresh HAL line markers after merging the review fixes

Co-Authored-By: Claude Opus 5.5 <noreply@anthropic.com>
Claude-Session: https://claude.ai/code/session_01KTrV7z7yWp6QksMj6bfNMx
Signed-off-by: Adrian <adrianllopart@gmail.com>

* fix(tools): refuse a --scene copy that differs from the committed scene

The OpenArm world-voxel wrapper checked only robot_id, the kernel's
world-voxel flag and robot_unit on a --scene copy, so a copy could turn
octomap off, widen the self-filter padding, add allowed collision pairs
or a safety envelope, swap drivers/HAL, or enable the grasp allowance
and still pass every gate. The copy must now parse to the committed
scene exactly, bar the top-level grasp_declaration; any other
difference is refused with its key paths.

Co-Authored-By: Claude Opus 5.5 <noreply@anthropic.com>
Signed-off-by: Adrian <adrianllopart@gmail.com>

* fix(tools): keep --scene operator copies in a gitignored scenes/deploy/local/

Copies under the tracked scenes/deploy/ broke
test_deploy_scene_registry_is_complete and dirtied the tree, and the
wrapper tests wrote their temp scenes there. The wrapper now accepts
--scene only under scenes/deploy/local/ (gitignored, still resolved
with readlink -f under the repo); the registry and load tests glob
non-recursively, so they already skip it. The wrapper tests write
their copies there and unlink them in finally.

Co-Authored-By: Claude Opus 5.5 <noreply@anthropic.com>
Signed-off-by: Adrian <adrianllopart@gmail.com>

* fix(reasoner): ground grasp contact links per hand, not per finger joint

The multi-gripper refusal only fired on an empty contact_links list and
counted role: gripper joints, so R1 Pro (four finger joints, two hands)
was refused as "4 grippers" and named links were never validated — a
link of the other hand, or a non-gripper link, went straight into the
GraspDeclaration.

gripper_hands() (replaces gripper_contact_links) groups the gripper
joints' child links by the arm they hang off (shared parent_link; a
chained finger joins its parent's hand). ground_grasp_target defaults an
empty list to the hand of a single-hand robot, refuses an empty list on
a multi-hand robot listing the hands, and refuses named links that are
not all gripper child links of one hand. Tests on the real openarm,
r1pro and so101 manifests.

Co-Authored-By: Claude Opus 5.5 <noreply@anthropic.com>
Claude-Session: https://claude.ai/code/session_01KTrV7z7yWp6QksMj6bfNMx
Signed-off-by: Adrian <adrianllopart@gmail.com>

* docs(core): say GraspDeclaration.search_box is a search hint, not the support plane

The docstring (and every generated JSON schema embedding it) still said
the box's bottom face is the support plane. The producer measures the
support layer from the voxel map and the reasoner pads the box downward
so that layer lies inside it; the box carries no support semantics.

Co-Authored-By: Claude Opus 5.5 <noreply@anthropic.com>
Claude-Session: https://claude.ai/code/session_01KTrV7z7yWp6QksMj6bfNMx
Signed-off-by: Adrian <adrianllopart@gmail.com>

* fix(reasoner): refuse grasp grounding without the deploy's voxel resolution

grasp_target_voxel_m defaulted to 0.02, a literal duplicating the real
cell's octree resolution that deploy_e2e already passes
(_octomap_resolution). A reasoner launched without it silently padded
every seed box by a cell size that may not be the map's. The default is
now 0.0 (unset) and grounding a grasp target with it unset raises
ROSReasonerInvalidPlan ("grasp grounding needs the deploy's voxel
resolution"), so no goal is sent.

Co-Authored-By: Claude Opus 5.5 <noreply@anthropic.com>
Claude-Session: https://claude.ai/code/session_01KTrV7z7yWp6QksMj6bfNMx
Signed-off-by: Adrian <adrianllopart@gmail.com>

* fix(hal): measure the grasp target's support as the surface ringing it

support_top_from_voxels took the highest layer holding half the densest
layer's count. In a tight detection column the table is mostly hidden
(under the item, in its shadow), so a 10x10 cm item's 25-cell top beat the
~35-cell visible table ring and became the "support": the producer never
seeded. The support is now the first layer, scanning down, whose
top-surface cells ring the footprint of the component standing above it
(between one cell and probe_margin_m out). A surface extends past what
stands on it; the target's own layers do not. The ring replaces the fixed
0.10 m support_cells_under square, which a target wider than ~20 cm covered
entirely (its cells are occluded), so it scales with the target.

Tests: occluded ring under a dense item top, a small item, an item on a
shelf board edge above a bench, plus the existing cell-scene cases.

Co-Authored-By: Claude Opus 5.5 <noreply@anthropic.com>
Claude-Session: https://claude.ai/code/session_01KTrV7z7yWp6QksMj6bfNMx
Signed-off-by: Adrian <adrianllopart@gmail.com>

* fix(hal): make the grasp target's support tunables constructor arguments

The support search depth (0.15 m) and the ring probe margin (0.05 m) were
module constants. They are calibration points that depend on the cell's
detector and camera, so GraspTargetLeg now takes them as
support_search_below_m / support_probe_margin_m with those defaults and
refuses non-positive values; the config fields can be wired by the
integrator without touching the leg. A 25x30 cm target, whose footprint
covered the old fixed 0.10 m probe square entirely, now finds the visible
table around it.

Co-Authored-By: Claude Opus 5.5 <noreply@anthropic.com>
Claude-Session: https://claude.ai/code/session_01KTrV7z7yWp6QksMj6bfNMx
Signed-off-by: Adrian <adrianllopart@gmail.com>

* fix(hal): refuse a grasp target that does not stand on the measured support

When a shelf board's exposed lip is hidden, the first surface ringing the
target can be a bench 10 cm below it. A region stood on that bench would
exempt the gap down to it (HZ-01xx-6). The seed cluster's lowest cell must
now sit within one voxel (the layer the seed drops) plus one voxel of
tolerance of the support, else a not_on_support contradiction and no
region. The seed is taken over the whole support column so a lifted search
box bottom cannot clip the target's lower cells from that check.

Co-Authored-By: Claude Opus 5.5 <noreply@anthropic.com>
Claude-Session: https://claude.ai/code/session_01KTrV7z7yWp6QksMj6bfNMx
Signed-off-by: Adrian <adrianllopart@gmail.com>

* fix(hal): hold an occluded grasp target only while the robot's hand is at it

The last round treated any re-fit inside the held region that failed the
map or tracking gate as the closing hand occluding the target, keeping the
exemption for the freeze TTL even when a person's hand or a knocked-away
target caused it — less conservative than before. Now a re-fit the map
does not cover is always map_disagrees (retract), and a covered re-fit
shrunk inside the held region is occluded_refit (freeze) only while a
declared contact link's tf origin lies within one voxel + occluder_margin_m
of the held region; otherwise it is unoccluded_refit and retracts at once.
GraspTargetLeg takes occluder_margin_m (default 0.05 m).

Co-Authored-By: Claude Opus 5.5 <noreply@anthropic.com>
Claude-Session: https://claude.ai/code/session_01KTrV7z7yWp6QksMj6bfNMx
Signed-off-by: Adrian <adrianllopart@gmail.com>

* fix(cli): judge the grasp-allowance producer refusal on the effective HAL params

`deploy run` refused `grasp_allowance_enabled` without the vision target leg by
reading the scene's `grasp_target_enabled`, so `--hal
vision_attachment_grasp_target_enabled=false` defeated it, and a bare
`ros2 launch deploy_e2e ... grasp_allowance_enabled:=true` was never checked.

The CLI now judges the merged HAL params (scene + `--hal`), and the launch reads
the HAL's params file back (`_hal_file_params`) and refuses the exemption on any
non-sim launch unless `enable_vision_attachment:=true` and the HAL file turns
the leg and its grasp-target producer on. The launch tests now write the real
params file the way `deploy` does.

Co-Authored-By: Claude Opus 5.5 <noreply@anthropic.com>
Signed-off-by: Adrian <adrianllopart@gmail.com>

* fix(launch): refuse vision-leg bounds that outrun the kernel's voxel path

`vision_attachment_grid_max_age_s` / `_release_clear_m` are derived from the
kernel's voxel deadline and margin + resolution, but the CLI's params file is
loaded after them, so any `--hal` or hand-written value won unchecked. The
launch now checks the effective value (derived merged with the HAL params file)
whenever the leg is on and fails with `ROSConfigError` for a grid age above
`world_voxel_deadline_s` or a release clearance below margin + one ce

File: robots/openarm/openarm.urdf (robot description, URDF)
Before this commit: robot openarm_v20, 22 links, 21 joints
Links:
- link openarm_left_base_link: mass 0.487784887988258 -> 1.1432284943239561
- link openarm_left_link1: mass 0.561428544234246 -> 1.1416684646202298
- link openarm_left_link2: mass 0.295592749115978 -> 0.2775092746011571
- link openarm_left_link3: mass 0.850916861288263 -> 1.073863338202347
- link openarm_left_link4: mass 0.590845933035621 -> 0.6348534566833373
- link openarm_left_link5: mass 0.5803968030561 -> 0.6156588026168502
- link openarm_left_link6: mass 0.368168327082267 -> 0.475202773187987
- link openarm_right_base_link: mass 0.487784887988258 -> 1.1432284943239561
- link openarm_right_link1: mass 0.561428544234246 -> 1.1416684646202298
- link openarm_right_link2: mass 0.295592749115978 -> 0.2775092746011571
- link openarm_right_link3: mass 0.850916861288263 -> 1.073863338202347
- link openarm_right_link4: mass 0.590845933035621 -> 0.6348534566833373
- link openarm_right_link5: mass 0.5803968030561 -> 0.6156588026168502
- link openarm_right_link6: mass 0.368168327082267 -> 0.475202773187987
Joints:
- joint openarm_left_finger_joint1: limit lower=-1.5708 upper=0 effort=7 velocity=5 -> lower=0 upper=1.5708 effort=7 velocity=5
- joint openarm_left_finger_joint2: limit lower=0 upper=1.5708 effort=7 velocity=5 -> lower=-1.5708 upper=0 effort=7 velocity=5
