Commit message: feat(robots): lower the DROID Franka + Robotiq self-collision model
`openral collision lower` refused robots/droid_franka_robotiq ("URDF produced
zero collision geometry"): its composed URDF named meshes package://, which
the lowering deliberately does not resolve. The URDF now uses the rd: form of
every other vendored URDF (panda_description / robotiq_2f85_v4_description
clones, the same pinned commits), so the two PUBLIC_ROS_PACKAGES entries added
for it are dropped again.

The manifest gains fixed_attachments panda_link7 -> panda_link8 ->
robotiq_arg2f_base_link (panda_joint8, robotiq_mount_joint) and the generated
collision_geometry (box + exact hull per link, as franka_panda) and sampled
ACM (adjacent arm pairs only). At the scenes' start pose
(0, -pi/5, 0, -4pi/5, 0, 3pi/5, 0, open) nothing trips; the nearest checked pair
is panda_link7 / robotiq_arg2f_base_link at 12.9 mm.

finger_joint's child is now the logical robotiq_finger_pair (franka_panda's
pattern): the kernel would have posed left_outer_knuckle at the normalised jaw
fraction read as radians, against the URDF's inverted 0..0.8 rad travel. The
jaw linkage therefore carries no primitive. Covering it with mimic links needs
safety-package work (the URDF lowering does not scope mimic_joints, and a
normalised leader has no radian mapping); recorded in KNOWN_GAPS and README.

The fleet guards cover the robot: drift (collision lowering fleet), URDF
enclosure, contact sweep, static-link audit, and the rest-pose check, which
now falls back to a deploy scene's initial_joint_positions when q = 0 is out
of limits and there is no SRDF.

Review the ACM with the Safety WG (CLAUDE.md §3).

Co-Authored-By: Claude Opus 5.5 <noreply@anthropic.com>
Claude-Session: https://claude.ai/code/session_011PRmh7XnocWrwny4cLo4r6
Signed-off-by: Adrian <adrianllopart@gmail.com>
(cherry picked from commit 58e3025d946cf018352f817be12e17e499853843)

File: robots/droid_franka_robotiq/droid_franka_robotiq.urdf (robot description, URDF)
Before this commit: robot droid_franka_robotiq, 19 links, 18 joints
Links:
- link left_bar: geometry collision mesh filename=rd:robotiq_2f85_v4_description:robotiq_2f_85_gripper_visual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; visual mesh filename=rd:robotiq_2f85_v4_description:robotiq_2f_85_gripper_visual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
- link left_distal_phalanx: geometry collision mesh filename=rd:robotiq_2f85_v4_description:robotiq_2f_85_gripper_visual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; visual mesh filename=rd:robotiq_2f85_v4_description:robotiq_2f_85_gripper_visual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
- link left_outer_knuckle: geometry collision mesh filename=rd:robotiq_2f85_v4_description:robotiq_2f_85_gripper_visual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; visual mesh filename=rd:robotiq_2f85_v4_description:robotiq_2f_85_gripper_visual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
- link left_proximal_phalanx: geometry collision mesh filename=rd:robotiq_2f85_v4_description:robotiq_2f_85_gripper_visual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; visual mesh filename=rd:robotiq_2f85_v4_description:robotiq_2f_85_gripper_visual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
- link panda_link0: geometry collision mesh filename=rd:panda_description:robots/panda_description/meshes/collis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; visual mesh filename=rd:panda_description:robots/panda_description/meshes/visual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
- link panda_link1: geometry collision mesh filename=rd:panda_description:robots/panda_description/meshes/collis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; visual mesh filename=rd:panda_description:robots/panda_description/meshes/visual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
- link panda_link2: geometry collision mesh filename=rd:panda_description:robots/panda_description/meshes/collis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; visual mesh filename=rd:panda_description:robots/panda_description/meshes/visual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
- link panda_link3: geometry collision mesh filename=rd:panda_description:robots/panda_description/meshes/collis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; visual mesh filename=rd:panda_description:robots/panda_description/meshes/visual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
- link panda_link4: geometry collision mesh filename=rd:panda_description:robots/panda_description/meshes/collis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; visual mesh filename=rd:panda_description:robots/panda_description/meshes/visual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
- link panda_link5: geometry collision mesh filename=rd:panda_description:robots/panda_description/meshes/collis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; visual mesh filename=rd:panda_description:robots/panda_description/meshes/visual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
- link panda_link6: geometry collision mesh filename=rd:panda_description:robots/panda_description/meshes/collis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; visual mesh filename=rd:panda_description:robots/panda_description/meshes/visual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
- link panda_link7: geometry collision mesh filename=rd:panda_description:robots/panda_description/meshes/collis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; visual mesh filename=rd:panda_description:robots/panda_description/meshes/visual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
- link right_bar: geometry collision mesh filename=rd:robotiq_2f85_v4_description:robotiq_2f_85_gripper_visual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; visual mesh filename=rd:robotiq_2f85_v4_description:robotiq_2f_85_gripper_visual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
- link right_distal_phalanx: geometry collision mesh filename=rd:robotiq_2f85_v4_description:robotiq_2f_85_gripper_visual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; visual mesh filename=rd:robotiq_2f85_v4_description:robotiq_2f_85_gripper_visual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
- link right_outer_knuckle: geometry collision mesh filename=rd:robotiq_2f85_v4_description:robotiq_2f_85_gripper_visual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; visual mesh filename=rd:robotiq_2f85_v4_description:robotiq_2f_85_gripper_visual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
- link right_proximal_phalanx: geometry collision mesh filename=rd:robotiq_2f85_v4_description:robotiq_2f_85_gripper_visual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; visual mesh filename=rd:robotiq_2f85_v4_description:robotiq_2f_85_gripper_visual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
- link robotiq_arg2f_base_link: geometry collision mesh filename=rd:robotiq_2f85_v4_description:robotiq_2f_85_gripper_visual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; visual mesh filename=rd:robotiq_2f85_v4_description:robotiq_2f_85_gripper_visual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
